File: _saved_CANtest IO Board.sch (KiCad schematic (older format))
At the start: 40 parts, among them J1 Inputs, J2 Conn_02x16_Counter_Clockwise, J3 Outputs, SW2 SW_SPST, SW3 SW_SPST, SW4 SW_Push, SW5 SW_Push

Commit message: Progress
Parts:
- removed SW2, SW3: SW_SPST, symbol SW_SPST
- added SW2, SW3: OS102011MS2QN1C, OS102011MS2QN1C:OS102011MS2QN1C, symbol OS102011MS2QN1C
- D1, D2, D3, D4, D5: footprint LEDs:LED_D3.0mm_Horizontal_O1.27mm_Z6.0mm -> LEDs:LED_D3.0mm
- D10, D11, D12, D13, D14, D15, D16, D6, D7, D8, D9: footprint LEDs:LED_Rectangular_W5.0mm_H2.0mm_Horizontal_O1.27mm_Z5.0mm -> LEDs:LED_Rectangular_W5.0mm_H2.0mm
- SW1: renamed from S?; footprint SHDR4W87P0X320_1X4_1511X584X1100P -> 1825117-1:SHDR4W87P0X320_1X4_1511X584X1100P
- SW4, SW5: footprint (none) -> Buttons_Switches_SMD:SW_SPST_KMR2
Connections:
- net IN3: now also SW2.1 (NO)
- net IN4: now also SW3.1 (NO)
- net VDD: now also SW2.2 (COM), SW3.2 (COM)
Other:
- moved on the sheet: SW4
