File: CANtest IO Board.kicad_pcb (KiCad board)
At the start: 2 copper layers, 40 parts, among them J1 Inputs, J2 Conn_02x16_Counter_Clockwise, J3 Outputs, SW1 1825117-1, SW2 OS102011MS2QN1C, SW3 OS102011MS2QN1C, SW4 SW_Push, SW5 SW_Push

Commit message: Progress2
Parts:
- added D17: LED, LEDs:LED_Rectangular_W5.0mm_H2.0mm, F.Cu at (130.8, 94.0)
- added D18: LED, LEDs:LED_Rectangular_W5.0mm_H2.0mm, F.Cu at (153.7, 91.4)
- added D19: LED, LEDs:LED_Rectangular_W5.0mm_H2.0mm, F.Cu at (153.7, 71.1)
- added D20: LED, LEDs:LED_Rectangular_W5.0mm_H2.0mm, F.Cu at (165.1, 68.6)
- added D21: LED, LEDs:LED_Rectangular_W5.0mm_H2.0mm, F.Cu at (165.1, 94.0)
- added R17: R, Resistors_SMD:R_0805_HandSoldering, F.Cu at (132.1, 96.5)
- added R18: R, Resistors_SMD:R_0805_HandSoldering, F.Cu at (154.9, 88.9)
- added R19: R, Resistors_SMD:R_0805_HandSoldering, F.Cu at (154.9, 68.6)
- added R20: R, Resistors_SMD:R_0805_HandSoldering, F.Cu at (166.4, 71.1)
- added R21: R, Resistors_SMD:R_0805_HandSoldering, F.Cu at (166.4, 96.5)
- moved D4 67.2 mm to (106.7, 85.1)
- moved D5 65.6 mm to (111.8, 85.1)
- moved R4 63.1 mm to (108.0, 82.5), turned to 180 degrees
- moved R5 61.9 mm to (113.0, 82.5), turned to 180 degrees
- moved D6 57.4 mm to (119.4, 91.4)
- moved D7 57.4 mm to (119.4, 94.0)
- moved R16 54.8 mm to (166.4, 63.5), turned to 180 degrees
- moved D10 54.3 mm to (142.2, 91.4)
- moved R6 54.0 mm to (120.7, 88.9), turned to 180 degrees
- moved R10 54.0 mm to (143.5, 88.9), turned to 180 degrees
- moved D8 52.2 mm to (130.8, 91.4)
- moved R13 52.2 mm to (143.5, 78.7), turned to 180 degrees
- moved R7 51.7 mm to (120.7, 96.5), turned to 180 degrees
- moved D13 50.3 mm to (142.2, 81.3)
- moved R8 50.3 mm to (132.1, 88.9), turned to 180 degrees
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