File: CANtest IO Board.sch (KiCad schematic (older format))
At the start: 40 parts, among them J1 Inputs, J2 Conn_02x16_Counter_Clockwise, J3 Outputs, SW1 SW_SPDT_MSM, SW2 SW_SPST, SW3 SW_SPST, SW4 SW_Push, SW5 SW_Push

Commit message: Progress
Parts:
- removed SW1: SW_SPDT_MSM, symbol SW_SPDT_MSM
- removed SW2, SW3: SW_SPST, symbol SW_SPST
- added SW1: 1825117-1, SHDR4W87P0X320_1X4_1511X584X1100P, symbol 1825117-1
- added SW2, SW3: OS102011MS2QN1C, OS102011MS2QN1C, symbol OS102011MS2QN1C
- D1, D2, D3, D4, D5: footprint (none) -> LEDs:LED_D3.0mm_Horizontal_O1.27mm_Z6.0mm
- D10, D11, D12, D13, D14, D15, D16, D6, D7, D8, D9: footprint (none) -> LEDs:LED_Rectangular_W5.0mm_H2.0mm_Horizontal_O1.27mm_Z5.0mm
- J1, J3: footprint (none) -> TerminalBlocks_Phoenix:TerminalBlock_Phoenix_MPT-2.54mm_9pol
- J2: footprint (none) -> Pin_Headers:Pin_Header_Angled_2x16_Pitch2.54mm
- R1, R10, R11, R12, R13, R14, R15, R16, R2, R3, R4, R5, R6, R7, R8, R9: footprint (none) -> Resistors_SMD:R_0805_HandSoldering
- SW4, SW5: footprint (none) -> Buttons_Switches_SMD:SW_SPST_KMR2
Connections:
- net IN1: now also SW1.1
- net IN2: now also SW1.4
- net IN3: now also SW2.1 (NO)
- net IN4: now also SW3.1 (NO)
- net VDD: now also SW1.2, SW1.3, SW2.2 (COM), SW3.2 (COM)
Other:
- moved on the sheet: SW4

Commit message: Progress2
Parts:
- added D17, D18, D19, D? (x2): LED, LEDs:LED_Rectangular_W5.0mm_H2.0mm, symbol LED
- added R17, R18, R19, R? (x2): R, Resistors_SMD:R_0805_HandSoldering, symbol R
- D1, D2, D3, D4, D5: footprint LEDs:LED_D3.0mm_Horizontal_O1.27mm_Z6.0mm -> LEDs:LED_D3.0mm
- D10, D11, D12, D13, D14, D15, D16, D6, D7, D8, D9: footprint LEDs:LED_Rectangular_W5.0mm_H2.0mm_Horizontal_O1.27mm_Z5.0mm -> LEDs:LED_Rectangular_W5.0mm_H2.0mm
- SW1: footprint SHDR4W87P0X320_1X4_1511X584X1100P -> 1825117-1:SHDR4W87P0X320_1X4_1511X584X1100P
- SW2, SW3: footprint OS102011MS2QN1C -> OS102011MS2QN1C:OS102011MS2QN1C
Connections:
- net GND: now also R17.1, R18.1, R19.1, R?.1, R?.1
- net OUT13: now also D?.2 (A)
- net OUT14: now also D17.2 (A)
- net OUT15: now also D?.2 (A)
- net OUT3: now also D19.2 (A)
- net OUT9: now also D18.2 (A)
- new net: D17.1 (K), R17.2
- new net: D19.1 (K), R19.2
- new net: D18.1 (K), R18.2
- new net: D?.1 (K), R?.2 (x2)
Other:
- moved on the sheet: D16, D8, R16, R8
